Commit message: fixed incorrect positioning of IMU, Lidar and Camera

File: src/mecanum_sim/nexus_4wd_mecanum_description/urdf/nexus_4wd_mecanum.xacro (robot description, xacro)
@@ -329,5 +329,5 @@
   <joint name="imu_joint" type="fixed">
     <axis xyz="0 1 0" />
-    <origin xyz="0.125 0 0.125" rpy="0 0 0"/>
+    <origin xyz="-0.15 0 0.025" rpy="0 0 0"/>
     <parent link="base_link"/>
     <child link="imu_link"/>
@@ -359,5 +359,5 @@
   <joint name="camera_joint" type="fixed">
     <axis xyz="0 1 0" />
-    <origin xyz="0.125 0 0.175" rpy="0 0 0"/>
+    <origin xyz="0.15 0 0.05" rpy="0 0 0"/>
     <parent link="base_link"/>
     <child link="camera_link"/>
@@ -388,5 +388,5 @@
    <!-- Hokuyo joint -->
   <joint name="hokuyo_joint" type="fixed">
-    <origin xyz="0.125 0.0 0.225" rpy="0 0 0"/>
+    <origin xyz="-0.15 0.0 0.075" rpy="0 0 0"/>
     <parent link="base_link"/>
     <axis xyz="0 1 0" />

Commit message: sample code

File: src/mecanum_sim/nexus_4wd_mecanum_description/urdf/nexus_4wd_mecanum.xacro (robot description, xacro)
@@ -359,5 +359,5 @@
   <joint name="camera_joint" type="fixed">
     <axis xyz="0 1 0" />
-    <origin xyz="0.15 0 0.05" rpy="0 0 0"/>
+    <origin xyz="0.15 0 0.05" rpy="0 -0.1 0"/>
     <parent link="base_link"/>
     <child link="camera_link"/>
@@ -458,5 +458,5 @@
       <update_rate>30.0</update_rate>
       <camera name="head">
-        <horizontal_fov>1.3962634</horizontal_fov>
+        <horizontal_fov>1.5962634</horizontal_fov>
         <image>
           <width>1920</width>
